File: sputterer.kicad_pcb (KiCad board)
At the start: 2 copper layers, 46 x 110 mm, 42 parts, among them J1 AudioJack2, J2 AudioJack2, J3 AudioJack2, J4 2X8 Header, J5 Conn_02x05_Odd_Even, Q1 BS170, U1 NE5532, U2 NE5532

Commit message: Changes to board and code
Parts:
- removed D5, D6: 1N4148, Diode_THT:D_DO-35_SOD27_P7.62mm_Horizontal
- added JP3: Conn_01x02_Male, Connector_PinHeader_2.54mm:PinHeader_1x02_P2.54mm_Vertical, F.Cu at (56.0, 154.2)
- LP1: footprint sputterer:LightPipe -> sputterizer:LightPipe
- RV1, RV2, RV3: footprint Potentiometer_THT:Potentiometer_Bourns_PTV09A-2_Single_Horizontal -> panel:Potentiometer_Bourns_PTD901_Single_Horizontal
- moved JP1 23.3 mm to (67.0, 109.5), turned to 90 degrees
- moved J4 18.2 mm to (56.0, 123.5), turned to 180 degrees
- moved R6 1.80 mm to (68.0, 106.0)
- turned JP2 to 180 degrees
Connections:
- A1 pad 30: Net-(A1-Pad30) -> +12V
- J4 pad 11: +5V -> Net-(J4-Pad11)
- J4 pad 12: +5V -> Net-(J4-Pad12)
Routing:
- net +12V: track 71.8 -> 116.6 mm, vias 2 -> 3
- net Net-(JP1-Pad2): track 56.3 -> 42.7 mm
- net /Gate: track 26.3 -> 38.4 mm, vias 1 -> 3
- net Net-(A1-Pad28): track 0.00 -> 7.63 mm, vias 0 -> 1
- net /CV: track 20.1 -> 14.1 mm, vias 1 -> 0
- net GND: track 15.9 -> 18.5 mm
- net Net-(A1-Pad8): track 103.1 -> 105.0 mm, vias 1 -> 2
- net Net-(A1-Pad7): track 102.0 -> 100.2 mm
- net Net-(C9-Pad1): track 20.5 -> 19.4 mm
- net +5V: track 0.00 -> 1.05 mm
- net -12V: track 76.7 -> 75.9 mm
- net Net-(C8-Pad1): track 12.5 -> 11.7 mm

Commit message: New design and code.
Parts:
- removed LP1: LightPipe, sputterizer:LightPipe
- moved D7 9.43 mm to (88.8, 153.0), turned to 90 degrees
Routing:
- net Net-(D7-Pad1): track 3.50 -> 12.9 mm
- net Net-(D7-Pad2): track 7.11 -> 12.9 mm
- net Net-(A1-Pad23): track 84.4 -> 83.9 mm
Changed lines of the file:
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@@
     (thickness 1.6)
     (drawings 10)
-    (tracks 303)
+    (tracks 300)
     (zones 0)
-    (modules 41)
+    (modules 40)
     (nets 48)
   )
@@
     (add_net "Net-(U1-Pad1)")
     (add_net "Net-(U2-Pad6)")
-  )
-  (module sputterizer:LightPipe (layer F.Cu)
-    (at 87.5 152)
-    (fp_text reference LP1 (at 0 2.465) (layer F.SilkS)
-      (effects (font (size 1 1) (thickness 0.15)))
-    )
-    (fp_text value LightPipe (at 0 -2.465) (layer F.Fab)
-      (effects (font (size 1 1) (thickness 0.15)))
-    )
-    (fp_line (start -7.72 0) (end -6 0) (layer F.SilkS) (width 0.12))
-    (fp_line (start -6.86 -1) (end -6.86 1) (layer F.SilkS) (width 0.12))
-    (fp_line (start 3 -1.5) (end 10 -1.5) (layer F.SilkS) (width 0.12))
-    (fp_line (start 10 -1.5) (end 10 1.5) (layer F.SilkS) (width 0.12))
-    (fp_line (start 10 1.5) (end 3 1.5) (layer F.SilkS) (width 0.12))
-    (fp_line (start -2.7 1.22) (end -2.7 -1.22) (layer F.CrtYd) (width 0.05))
-    (fp_line (start 2.7 1.22) (end -2.7 1.22) (layer F.CrtYd) (width 0.05))
-    (fp_line (start 2.7 -1.22) (end 2.7 1.22) (layer F.CrtYd) (width 0.05))
-    (fp_line (start -2.7 -1.22) (end 2.7 -1.22) (layer F.CrtYd) (width 0.05))
-    (fp_line (start 0 -1.465) (end 0 1.465) (layer F.SilkS) (width 0.12))
-    (fp_line (start -2.95 1.465) (end -2.95 -1.465) (layer F.SilkS) (width 0.12))
-    (fp_line (start 2.95 1.465) (end -2.95 1.465) (layer F.SilkS) (width 0.12))
-    (fp_line (start 2.95 -1.465) (end 2.95 1.465) (layer F.SilkS) (width 0.12))
-    (fp_line (start -2.95 -1.465) (end 2.95 -1.465) (layer F.SilkS) (width 0.12))
-    (pad 2 thru_hole circle (at 1.485 0) (size 2 2) (drill 2) (layers *.Cu *.Mask))
-    (pad 1 thru_hole circle (at -1.485 0) (size 2 2) (drill 2) (layers *.Cu *.Mask))
   )
   (module Connector_PinHeader_2.54mm:PinHeader_2x05_P2.54mm_Vertical (layer F.Cu)
@@
   )
   (module LED_THT:LED_D3.0mm (layer F.Cu)
-    (at 79.375 152)
+    (at 88.75 153 90)
     (descr "LED, diameter 3.0mm, 2 pins")
     (tags "LED diameter 3.0mm 2 pins")
-    (fp_text reference D7 (at 1.27 -2.96) (layer F.SilkS)
-      (effects (font (size 1 1) (thickness 0.15)))
-    )
-    (fp_text value LED (at 1.27 2.96) (layer F.Fab)
+    (fp_text reference D7 (at 1.27 3.5) (layer F.SilkS)
+      (effects (font (size 1 1) (thickness 0.15)))
+    )
+    (fp_text value LED (at 1.27 2.96 90) (layer F.Fab)
       (effects (font (size 1 1) (thickness 0.15)))
     )
@@
     (fp_arc (start 1.27 0) (end -0.29 -1.235516) (angle 108.8) (layer F.SilkS) (width 0.12))
     (fp_arc (start 1.27 0) (end -0.23 -1.16619) (angle 284.3) (layer F.Fab) (width 0.1))
-    (pad 2 thru_hole circle (at 2.54 0) (size 1.8 1.8) (drill 0.9) (layers *.Cu *.Mask)
+    (pad 2 thru_hole circle (at 2.54 0 90) (size 1.8 1.8) (drill 0.9) (layers *.Cu *.Mask)
       (net 36 "Net-(D7-Pad2)"))
-    (pad 1 thru_hole rect (at 0 0) (size 1.8 1.8) (drill 0.9) (layers *.Cu *.Mask)
+    (pad 1 thru_hole rect (at 0 0 90) (size 1.8 1.8) (drill 0.9) (layers *.Cu *.Mask)
       (net 35 "Net-(D7-Pad1)"))
     (model ${KISYS3DMOD}/LED_THT.3dshapes/LED_D3.0mm.wrl
@@
   (segment (start 60.12 131.5) (end 59.62 131) (width 0.25) (layer F.Cu) (net 13))
   (segment (start 66.84 131.5) (end 60.12 131.5) (width 0.25) (layer F.Cu) (net 13))
-  (segment (start 87.105001 157.394999) (end 87.105001 158.894999) (width 0.25) (layer B.Cu) (net 14))
-  (segment (start 87.5 157) (end 87.105001 157.394999) (width 0.25) (layer B.Cu) (net 14))
-  (segment (start 87.105001 158.894999) (end 87 159) (width 0.25) (layer B.Cu) (net 14))
-  (segment (start 87 159) (end 87 159.5) (width 0.25) (layer B.Cu) (net 14))
   (segment (start 87 159.5) (end 87 159.5) (width 0.25) (layer B.Cu) (net 14))
-  (via (at 87 159.5) (size 0.8) (drill 0.4) (layers F.Cu B.Cu) (net 14))
+  (via (at 87.25 159.5) (size 0.8) (drill 0.4) (layers F.Cu B.Cu) (net 14))
   (segment (start 75.02 159.5) (end 73.28 157.76) (width 0.25) (layer F.Cu) (net 14))
   (segment (start 87 159.5) (end 75.02 159.5) (width 0.25) (layer F.Cu) (net 14))
-  (segment (start 87.5 93.227208) (end 87.5 123) (width 0.25) (layer B.Cu) (net 14))
-  (segment (start 88.727208 92) (end 87.5 93.227208) (width 0.25) (layer B.Cu) (net 14))
+  (segment (start 88.727208 92) (end 87.25 93.227208) (width 0.25) (layer B.Cu) (net 14))
   (segment (start 90 92) (end 88.727208 92) (width 0.25) (layer B.Cu) (net 14))
-  (segment (start 87.5 122.5) (end 87.5 123) (width 0.25) (layer B.Cu) (net 14))
-  (segment (start 87.5 123) (end 87.5 157) (width 0.25) (layer B.Cu) (net 14))
+  (segment (start 87.25 157.25) (end 87.25 159.5) (width 0.25) (layer B.Cu) (net 14))
+  (segment (start 87.25 93.227208) (end 87.25 157.25) (width 0.25) (layer B.Cu) (net 14))
   (via (at 50.5 169) (size 0.8) (drill 0.4) (layers F.Cu B.Cu) (net 15))
   (segment (start 69.194999 168.914999) (end 73.28 173) (width 0.25) (layer F.Cu) (net 15))
@@
   (segment (start 72 87.5) (end 73.5 89) (width 0.25) (layer B.Cu) (net 26))
   (segment (start 73.5 109) (end 73.5 129.5) (width 0.25) (layer B.Cu) (net 26))
-  (segment (start 84.724999 169.204999) (end 88.52 173) (width 0.25) (layer B.Cu) (net 26))
-  (segment (start 84.724999 150.224999) (end 84.724999 169.204999) (width 0.25) (layer B.Cu) (net 26))
-  (segment (start 83 129.5) (end 83 148.5) (width 0.25) (layer B.Cu) (net 26))
-  (segment (start 83 148.5) (end 84.724999 150.224999) (width 0.25) (layer B.Cu) (net 26))
+  (segment (start 83 148.5) (end 83 129.5) (width 0.25) (layer B.Cu) (net 26))
+  (segment (start 83 149) (end 83 148.5) (width 0.25) (layer B.Cu) (net 26))
+  (segment (start 84.724999 150.724999) (end 83 149) (width 0.25) (layer B.Cu) (net 26))
+  (segment (start 88.52 173) (end 84.724999 169.204999) (width 0.25) (layer B.Cu) (net 26))
+  (segment (start 84.724999 169.204999) (end 84.724999 150.724999) (width 0.25) (layer B.Cu) (net 26))
   (segment (start 61.62 137) (end 66.84 137) (width 0.25) (layer F.Cu) (net 28))
   (segment (start 59.62 139) (end 61.62 137) (width 0.25) (layer F.Cu) (net 28))
@@
   (segment (start 77 91) (end 79.66 91) (width 0.25) (layer F.Cu) (net 34))
   (segment (start 81 87.5) (end 81 92.34) (width 0.25) (layer B.Cu) (net 34))
-  (segment (start 76 152) (end 79.5 152) (width 0.25) (layer F.Cu) (net 35))
-  (segment (start 82 152) (end 82.04 152) (width 0.25) (layer F.Cu) (net 36))
-  (segment (start 77 147) (end 82 152) (width 0.25) (layer F.Cu) (net 36))
+  (segment (start 87.5 152) (end 88.5 153) (width 0.25) (layer F.Cu) (net 35))
+  (segment (start 76 152) (end 87.5 152) (width 0.25) (layer F.Cu) (net 35))
+  (segment (start 80.46 150.46) (end 88.5 150.46) (width 0.25) (layer F.Cu) (net 36))
+  (segment (start 77 147) (end 80.46 150.46) (width 0.25) (layer F.Cu) (net 36))
   (segment (start 87.6 126.5) (end 90.6 123.5) (width 0.25) (layer F.Cu) (net 37))
   (segment (start 77.16 126.5) (end 87.6 126.5) (width 0.25) (layer F.Cu) (net 37))
