File: front panel/panel/panel.kicad_pcb (KiCad board)
At the start: 2 copper layers, 55 x 128.5 mm, 25 parts

Commit message: Latest changes.
Other:
- board text added: "Maytag"
- board text added: "Toggle"
- board text added: "User"
- board text removed: "User 1"
- board text removed: "User 2"
- board text removed: "User 3"
Changed lines of the file:
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@@
     (effects (font (size 2 2) (thickness 0.25)))
   )
-  (gr_text "User 3" (at 74.5 159.5) (layer F.SilkS)
+  (gr_text User (at 72.5 159.5) (layer F.SilkS)
     (effects (font (size 2 2) (thickness 0.25)))
   )
-  (gr_text "User 2" (at 74.5 152.5) (layer F.SilkS)
+  (gr_text Maytag (at 74.5 152.5) (layer F.SilkS)
     (effects (font (size 2 2) (thickness 0.25)))
   )
-  (gr_text "User 1" (at 74.5 145.5) (layer F.SilkS)
+  (gr_text Toggle (at 74.5 145.5) (layer F.SilkS)
     (effects (font (size 2 2) (thickness 0.25)))
   )

Commit message: Changes to board and code
Parts:
- added H26: MountingHole, MountingHole:MountingHole_3.2mm_M3, F.Cu at (64.0, 73.5)
- added H27: MountingHole, MountingHole:MountingHole_3.2mm_M3, F.Cu at (91.0, 175.5)
- added H28: MountingHole, MountingHole:MountingHole_3.2mm_M3, F.Cu at (64.0, 175.5)
- added H29: MountingHole, MountingHole:MountingHole_3.2mm_M3, F.Cu at (91.0, 73.5)
- H1, H2, H3: footprint MountingHole:MountingHole_6.5mm -> panel:MountingHole_7.3mm
- moved H1 3.50 mm to (105.5, 79.0)
- moved H2 3.50 mm to (105.5, 96.5)
- moved H3 3.50 mm to (105.5, 113.5)
- moved H10 1.45 mm to (63.8, 89.5)
- moved H11 1.45 mm to (63.8, 96.5)
- moved H12 1.45 mm to (63.8, 103.5)
- moved H13 1.45 mm to (63.8, 110.5)
- moved H14 1.45 mm to (63.8, 117.5)
- moved H15 1.45 mm to (63.8, 124.5)
- moved H16 1.45 mm to (63.8, 131.5)
- moved H17 1.45 mm to (63.8, 138.5)
- moved H18 1.45 mm to (63.8, 145.5)
- moved H19 1.45 mm to (63.8, 152.5)
- moved H20 1.45 mm to (63.8, 159.5)
- moved H9 1.45 mm to (63.8, 82.5)
Other:
- board text added: "SELECT"
- board text removed: "Select"

Commit message: Latest checkin
Parts:
- added ?: , , F.Cu at (111.0, 95.5)
